Commit message: added changes to urdf and timing to ikPlanner etc.

File: src/ur5_rabot/ur5_with_sr300_support/urdf/ur5.urdf.xacro (robot description, xacro)
@@ -283,8 +283,8 @@
           <box size="0.03 0.12 0.03"/>
         </geometry>
-        <origin rpy="0 0 0" xyz="0.025 0 0"/>
+        <origin rpy="0 0 0" xyz="0.045 0 0.035"/>
       </collision>
 			<visual>
-      	<origin xyz="0.025 0 0" rpy="0 0 0"/>
+      	<origin xyz="0.045 0 0.035" rpy="0 0 0"/>
       	<geometry>
     	<box size="0.03 0.12 0.03"/>

Commit message: fixed joint limited launch files.. etc

File: src/ur5_rabot/ur5_with_sr300_support/urdf/ur5.urdf.xacro (robot description, xacro)
@@ -276,17 +276,17 @@
       <parent link="${prefix}wrist_3_link" />
       <child link = "${prefix}ee_link" />
-      <origin xyz="0.0 ${wrist_3_length} 0.0" rpy="0.0 0.0 ${pi/2.0}" />
+      <origin xyz="0.0 ${wrist_3_length} 0.0" rpy=" ${-pi/2} 0.0 0.0" />
     </joint>
     <link name="${prefix}ee_link">
       <collision>
         <geometry>
-          <box size="0.03 0.12 0.03"/>
-        </geometry>
-        <origin rpy="0 0 0" xyz="0.045 0 0.035"/>
+          <box size="0.12 0.3 0.03"/>
+        </geometry>
+        <origin xyz="0.0 -0.035 0.045" rpy="0 0 0"/>
       </collision>
 			<visual>
-      	<origin xyz="0.045 0 0.035" rpy="0 0 0"/>
+      	<origin xyz="0.0 -0.035 0.045" rpy="0 0 0"/>
       	<geometry>
-    	<box size="0.03 0.12 0.03"/>
+    	<box size="0.12 0.03 0.03"/>
       	</geometry>
       	<material name="red"/>
