Commit message: wut

File: src/ur5_rabot/ur5_with_sr300_support/urdf/ur5.urdf (robot description, URDF)
Before this commit: robot ur5, 11 links, 10 joints
Links:
- added link sensor; collision box size=0.03 0.12 0.03; visual box size=0.03 0.12 0.03
- added link tool_tip
- link ee_link: geometry collision box size=0.01 0.01 0.01
Joints:
- added joint tool_to_torch: type fixed, parent ee_link, child sensor
- added joint torch_to_tip: type fixed, parent sensor, child tool_tip, origin xyz=0.0 0.0 0.01 rpy=0 0.0 0
- joint elbow_joint: limit lower=-6.2831853 upper=6.2831853 effort=150.0 velocity=3.15 -> lower=-3.14159265 upper=3.14159265 effort=150.0 velocity=3.15
- joint shoulder_lift_joint: limit lower=-6.2831853 upper=6.2831853 effort=150.0 velocity=3.15 -> lower=-3.14159265 upper=3.14159265 effort=150.0 velocity=3.15
- joint shoulder_pan_joint: limit lower=-6.2831853 upper=6.2831853 effort=150.0 velocity=3.15 -> lower=-3.14159265 upper=3.14159265 effort=150.0 velocity=3.15
- joint wrist_1_joint: limit lower=-6.2831853 upper=6.2831853 effort=28.0 velocity=3.2 -> lower=-3.14159265 upper=3.14159265 effort=28.0 velocity=3.2
- joint wrist_2_joint: limit lower=-6.2831853 upper=6.2831853 effort=28.0 velocity=3.2 -> lower=-3.14159265 upper=3.14159265 effort=28.0 velocity=3.2
- joint wrist_3_joint: limit lower=-6.2831853 upper=6.2831853 effort=28.0 velocity=3.2 -> lower=-3.14159265 upper=3.14159265 effort=28.0 velocity=3.2

File: src/ur5_rabot/ur5_with_sr300_support/urdf/ur5.urdf.xacro (robot description, xacro)
@@ -276,20 +276,13 @@
       <parent link="${prefix}wrist_3_link" />
       <child link = "${prefix}ee_link" />
-      <origin xyz="0.0 ${wrist_3_length} 0.0" rpy=" ${-pi/2} 0.0 0.0" />
+      <origin xyz="0.0 ${wrist_3_length} 0.0" rpy="0.0 0.0 ${pi/2.0}" />
     </joint>
     <link name="${prefix}ee_link">
       <collision>
         <geometry>
-          <box size="0.12 0.3 0.03"/>
-        </geometry>
-        <origin xyz="0.0 -0.035 0.045" rpy="0 0 0"/>
-      </collision>
-			<visual>
-      	<origin xyz="0.0 -0.035 0.045" rpy="0 0 0"/>
-      	<geometry>
-    	<box size="0.12 0.03 0.03"/>
-      	</geometry>
-      	<material name="red"/>
-    	</visual>
+          <box size="0.01 0.01 0.01"/>
+        </geometry>
+        <origin rpy="0 0 0" xyz="-0.01 0 0"/>
+      </collision>
     </link>
     <xacro:ur_arm_transmission prefix="${prefix}" />

File: src/ur5_rabot/ur5_with_sr300_support/urdf/ur5_joint_limited_robot.urdf.xacro (robot description, xacro)
@@ -14,3 +14,28 @@
     <origin xyz="0.0 0.0 0.0" rpy="0.0 0.0 0.0" />
   </joint>
+<link name="sensor">
+ 	<visual>
+    <origin xyz="0.045 0.0 0.035" rpy="0 0.0 0.0" />
+  	<geometry>
+      <box size="0.03 0.12 0.03"/>
+     </geometry>
+     <material name="Grey" />
+ </visual>
+ <collision>
+    <origin xyz="0.045 0.0 0.35" rpy="0 0 0" />
+    <geometry>
+      <box size="0.03 0.12 0.03"/>
+    </geometry>
+ </collision>
+	</link>
+<link name="tool_tip" />
+<joint name="tool_to_sensor" type="fixed">
+  <parent link="ee_link"/>
+  <child link="sensor"/>
+</joint>
+<joint name="sensor_to_tip" type="fixed">
+  <parent link="sensor"/>
+  <child link="tool_tip"/>
+  <origin xyz="0.0 0.0 0.01" rpy="0 0.0 0" />
+</joint>
 </robot>

File: src/ur5_rabot/ur5_with_sr300_support/urdf/ur5_robot.urdf.xacro (robot description, xacro)
@@ -14,3 +14,28 @@
     <origin xyz="0.0 0.0 0.0" rpy="0.0 0.0 0.0" />
   </joint>
+	<link name="sensor">
+ 	<visual>
+    <origin xyz="0.045 0.0 0.035" rpy="0 0.0 0.0" />
+  	<geometry>
+      <box size="0.03 0.12 0.03"/>
+     </geometry>
+     <material name="Grey" />
+ </visual>
+ <collision>
+    <origin xyz="0.045 0.0 0.35" rpy="0 0 0" />
+    <geometry>
+      <box size="0.03 0.12 0.03"/>
+    </geometry>
+ </collision>
+	</link>
+<link name="tool_tip" />
+<joint name="tool_to_sensor" type="fixed">
+  <parent link="ee_link"/>
+  <child link="sensor"/>
+</joint>
+<joint name="sensor_to_tip" type="fixed">
+  <parent link="sensor"/>
+  <child link="tool_tip"/>
+  <origin xyz="0.0 0.0 0.01" rpy="0 0.0 0" />
+</joint>
 </robot>
